Commit message: hmm

File: src/prototype_description/urdf/prototype.xacro (robot description, xacro)
@@ -2,5 +2,5 @@
 <robot name="prototype" xmlns:xacro="http://www.ros.org/wiki/xacro">
 <xacro:include filename="$(find prototype_description)/urdf/materials.xacro" />
-<xacro:include filename="$(find prototype_description)/urdf/prototype.trans" />
+<xacro:include filename="$(find prototype_description)/urdf/prototype.ros2control" />
 <xacro:include filename="$(find prototype_description)/urdf/prototype.gazebo" />
 <link name="base_link">
@@ -33,5 +33,5 @@
     <origin xyz="0.287891 -0.110458 -0.0294" rpy="0 0 0"/>
     <geometry>
-      <mesh filename="file://$(find prototype_description)/meshes/stellarhd-wetlink_1.stl" scale="0.001 0.001 0.001"/>
+      <mesh filename="file://$(find prototype_description)/meshes/stellarhd-wetlink.stl" scale="0.001 0.001 0.001"/>
     </geometry>
     <material name="silver"/>
@@ -40,5 +40,5 @@
     <origin xyz="0.287891 -0.110458 -0.0294" rpy="0 0 0"/>
     <geometry>
-      <mesh filename="file://$(find prototype_description)/meshes/stellarhd-wetlink_1.stl" scale="0.001 0.001 0.001"/>
+      <mesh filename="file://$(find prototype_description)/meshes/stellarhd-wetlink.stl" scale="0.001 0.001 0.001"/>
     </geometry>
   </collision>
@@ -53,5 +53,5 @@
     <origin xyz="0.294041 -0.110458 -0.00315" rpy="0 0 0"/>
     <geometry>
-      <mesh filename="file://$(find prototype_description)/meshes/stellarhd-bracket_1.stl" scale="0.001 0.001 0.001"/>
+      <mesh filename="file://$(find prototype_description)/meshes/stellarhd-bracket.stl" scale="0.001 0.001 0.001"/>
     </geometry>
     <material name="silver"/>
@@ -60,5 +60,5 @@
     <origin xyz="0.294041 -0.110458 -0.00315" rpy="0 0 0"/>
     <geometry>
-      <mesh filename="file://$(find prototype_description)/meshes/stellarhd-bracket_1.stl" scale="0.001 0.001 0.001"/>
+      <mesh filename="file://$(find prototype_description)/meshes/stellarhd-bracket.stl" scale="0.001 0.001 0.001"/>
     </geometry>
   </collision>
@@ -73,5 +73,5 @@
     <origin xyz="0.579463 -0.579463 -0.0" rpy="0 0 0"/>
     <geometry>
-      <mesh filename="file://$(find prototype_description)/meshes/left_Aerial_Truss_Structure3_1.stl" scale="0.001 0.001 0.001"/>
+      <mesh filename="file://$(find prototype_description)/meshes/left_Aerial_Truss_Structure3.stl" scale="0.001 0.001 0.001"/>
     </geometry>
     <material name="silver"/>
@@ -80,5 +80,5 @@
     <origin xyz="0.579463 -0.579463 -0.0" rpy="0 0 0"/>
     <geometry>
-      <mesh filename="file://$(find prototype_description)/meshes/left_Aerial_Truss_Structure3_1.stl" scale="0.001 0.001 0.001"/>
+      <mesh filename="file://$(find prototype_description)/meshes/left_Aerial_Truss_Structure3.stl" scale="0.001 0.001 0.001"/>
     </geometry>
   </collision>
@@ -93,5 +93,5 @@
     <origin xyz="0.039519 -0.038944 -0.00315" rpy="0 0 0"/>
     <geometry>
-      <mesh filename="file://$(find prototype_description)/meshes/right_Aerial_Truss_Structure3_1.stl" scale="0.001 0.001 0.001"/>
+      <mesh filename="file://$(find prototype_description)/meshes/right_Aerial_Truss_Structure3.stl" scale="0.001 0.001 0.001"/>
     </geometry>
     <material name="silver"/>
@@ -100,5 +100,5 @@
     <origin xyz="0.039519 -0.038944 -0.00315" rpy="0 0 0"/>
     <geometry>
-      <mesh filename="file://$(find prototype_description)/meshes/right_Aerial_Truss_Structure3_1.stl" scale="0.001 0.001 0.001"/>
+      <mesh filename="file://$(find prototype_description)/meshes/right_Aerial_Truss_Structure3.stl" scale="0.001 0.001 0.001"/>
     </geometry>
   </collision>
@@ -113,5 +113,5 @@
     <origin xyz="0.442491 -0.0 -0.001575" rpy="0 0 0"/>
     <geometry>
-      <mesh filename="file://$(find prototype_description)/meshes/electronics_box_1.stl" scale="0.001 0.001 0.001"/>
+      <mesh filename="file://$(find prototype_description)/meshes/electronics_box.stl" scale="0.001 0.001 0.001"/>
     </geometry>
     <material name="silver"/>
@@ -120,5 +120,5 @@
     <origin xyz="0.442491 -0.0 -0.001575" rpy="0 0 0"/>
     <geometry>
-      <mesh filename="file://$(find prototype_description)/meshes/electronics_box_1.stl" scale="0.001 0.001 0.001"/>
+      <mesh filename="file://$(find prototype_description)/meshes/electronics_box.stl" scale="0.001 0.001 0.001"/>
     </geometry>
   </collision>
@@ -133,5 +133,5 @@
     <origin xyz="0.123682 -0.011712 -0.001575" rpy="0 0 0"/>
     <geometry>
-      <mesh filename="file://$(find prototype_description)/meshes/right_roll_servo_1.stl" scale="0.001 0.001 0.001"/>
+      <mesh filename="file://$(find prototype_description)/meshes/right_roll_servo.stl" scale="0.001 0.001 0.001"/>
     </geometry>
     <material name="silver"/>
@@ -140,5 +140,5 @@
     <origin xyz="0.123682 -0.011712 -0.001575" rpy="0 0 0"/>
     <geometry>
-      <mesh filename="file://$(find prototype_description)/meshes/right_roll_servo_1.stl" scale="0.001 0.001 0.001"/>
+      <mesh filename="file://$(find prototype_description)/meshes/right_roll_servo.stl" scale="0.001 0.001 0.001"/>
     </geometry>
   </collision>
@@ -153,5 +153,5 @@
     <origin xyz="0.101182 0.000788 -0.001575" rpy="0 0 0"/>
     <geometry>
-      <mesh filename="file://$(find prototype_description)/meshes/right_pitch_servo_1.stl" scale="0.001 0.001 0.001"/>
+      <mesh filename="file://$(find prototype_description)/meshes/right_pitch_servo.stl" scale="0.001 0.001 0.001"/>
     </geometry>
     <material name="silver"/>
@@ -160,5 +160,5 @@
     <origin xyz="0.101182 0.000788 -0.001575" rpy="0 0 0"/>
     <geometry>
-      <mesh filename="file://$(find prototype_description)/meshes/right_pitch_servo_1.stl" scale="0.001 0.001 0.001"/>
+      <mesh filename="file://$(find prototype_description)/meshes/right_pitch_servo.stl" scale="0.001 0.001 0.001"/>
     </geometry>
   </collision>
@@ -173,5 +173,5 @@
     <origin xyz="0.168363 0.016213 0.004387" rpy="0 0 0"/>
     <geometry>
-      <mesh filename="file://$(find prototype_description)/meshes/right_pitch_FRX430-H105K_1.stl" scale="0.001 0.001 0.001"/>
+      <mesh filename="file://$(find prototype_description)/meshes/right_pitch_FRX430-H105K.stl" scale="0.001 0.001 0.001"/>
     </geometry>
     <material name="silver"/>
@@ -180,5 +180,5 @@
     <origin xyz="0.168363 0.016213 0.004387" rpy="0 0 0"/>
     <geometry>
-      <mesh filename="file://$(find prototype_description)/meshes/right_pitch_FRX430-H105K_1.stl" scale="0.001 0.001 0.001"/>
+      <mesh filename="file://$(find prototype_description)/meshes/right_pitch_FRX430-H105K.stl" scale="0.001 0.001 0.001"/>
     </geometry>
   </collision>
@@ -193,5 +193,5 @@
     <origin xyz="0.4943 -0.011712 -0.001575" rpy="0 0 0"/>
     <geometry>
-      <mesh filename="file://$(find prototype_description)/meshes/left_pitch_servo_1.stl" scale="0.001 0.001 0.001"/>
+      <mesh filename="file://$(find prototype_description)/meshes/left_pitch_servo.stl" scale="0.001 0.001 0.001"/>
     </geometry>
     <material name="silver"/>
@@ -200,5 +200,5 @@
     <origin xyz="0.4943 -0.011712 -0.001575" rpy="0 0 0"/>
     <geometry>
-      <mesh filename="file://$(find prototype_description)/meshes/left_pitch_servo_1.stl" scale="0.001 0.001 0.001"/>
+      <mesh filename="file://$(find prototype_description)/meshes/left_pitch_servo.stl" scale="0.001 0.001 0.001"/>
     </geometry>
   </collision>
@@ -213,5 +213,5 @@
     <origin xyz="0.5153 0.000788 -0.001575" rpy="0 0 0"/>
     <geometry>
-      <mesh filename="file://$(find prototype_description)/meshes/left_FRX430-S105K_1.stl" scale="0.001 0.001 0.001"/>
+      <mesh filename="file://$(find prototype_description)/meshes/left_FRX430-S105K.stl" scale="0.001 0.001 0.001"/>
     </geometry>
     <material name="silver"/>
@@ -220,5 +220,5 @@
     <origin xyz="0.5153 0.000788 -0.001575" rpy="0 0 0"/>
     <geometry>
-      <mesh filename="file://$(find prototype_description)/meshes/left_FRX430-S105K_1.stl" scale="0.001 0.001 0.001"/>
+      <mesh filename="file://$(find prototype_description)/meshes/left_FRX430-S105K.stl" scale="0.001 0.001 0.001"/>
     </geometry>
   </collision>
@@ -233,5 +233,5 @@
     <origin xyz="0.5168 0.000788 -0.001575" rpy="0 0 0"/>
     <geometry>
-      <mesh filename="file://$(find prototype_description)/meshes/left_roll_servo_1.stl" scale="0.001 0.001 0.001"/>
+      <mesh filename="file://$(find prototype_description)/meshes/left_roll_servo.stl" scale="0.001 0.001 0.001"/>
     </geometry>
     <material name="silver"/>
@@ -240,5 +240,5 @@
     <origin xyz="0.5168 0.000788 -0.001575" rpy="0 0 0"/>
     <geometry>
-      <mesh filename="file://$(find prototype_description)/meshes/left_roll_servo_1.stl" scale="0.001 0.001 0.001"/>
+      <mesh filename="file://$(find prototype_description)/meshes/left_roll_servo.stl" scale="0.001 0.001 0.001"/>
     </geometry>
   </collision>
@@ -253,5 +253,5 @@
     <origin xyz="-0.034 0.016213 -0.007537" rpy="0 0 0"/>
     <geometry>
-      <mesh filename="file://$(find prototype_description)/meshes/left_FRX430-H105K_1.stl" scale="0.001 0.001 0.001"/>
+      <mesh filename="file://$(find prototype_description)/meshes/left_FRX430-H105K.stl" scale="0.001 0.001 0.001"/>
     </geometry>
     <material name="silver"/>
@@ -260,5 +260,5 @@
     <origin xyz="-0.034 0.016213 -0.007537" rpy="0 0 0"/>
     <geometry>
-      <mesh filename="file://$(find prototype_description)/meshes/left_FRX430-H105K_1.stl" scale="0.001 0.001 0.001"/>
+      <mesh filename="file://$(find prototype_description)/meshes/left_FRX430-H105K.stl" scale="0.001 0.001 0.001"/>
     </geometry>
   </collision>
@@ -273,5 +273,5 @@
     <origin xyz="0.102682 0.000788 -0.001575" rpy="0 0 0"/>
     <geometry>
-      <mesh filename="file://$(find prototype_description)/meshes/right_FRX430-S105K_1.stl" scale="0.001 0.001 0.001"/>
+      <mesh filename="file://$(find prototype_description)/meshes/right_FRX430-S105K.stl" scale="0.001 0.001 0.001"/>
     </geometry>
     <material name="silver"/>
@@ -280,5 +280,5 @@
     <origin xyz="0.102682 0.000788 -0.001575" rpy="0 0 0"/>
     <geometry>
-      <mesh filename="file://$(find prototype_description)/meshes/right_FRX430-S105K_1.stl" scale="0.001 0.001 0.001"/>
+      <mesh filename="file://$(find prototype_description)/meshes/right_FRX430-S105K.stl" scale="0.001 0.001 0.001"/>
     </geometry>
   </collision>
